File: framework16-m2-cellular.kicad_sch (KiCad schematic)
At the start: 92 parts, among them J1 M.2 Socket B-Key (2199230-3), J10 MHF4L (20579-001E), J11 SIM Card, J12 Fan 1, J13 Fan 2, J2 MHF4L (20579-001E), J3 MHF4L (20579-001E), J5 MHF4L (20579-001E), J6 MHF4L (20579-001E), J7 MHF4L (20579-001E)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

Commit message: Swap out capacitors with more low profile ones
Parts:
- C13, C5: LCSC C72494 -> C22383609
Changed lines of the file:
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@@
 			)
 		)
-		(property "LSCS" ""
-			(at 358.14 36.83 0)
-			(effects
-				(font
-					(size 1.27 1.27)
-				)
-				(hide yes)
-			)
-		)
-		(property "LCSC" "C72494"
+		(property "LCSC" "C22383609"
 			(at 358.14 36.83 0)
 			(effects
@@
 			)
 		)
-		(property "LSCS" ""
+		(property "LCSC" "C22383609"
 			(at 378.46 55.88 0)
 			(effects
-				(font
-					(size 1.27 1.27)
-				)
-				(hide yes)
-			)
-		)
-		(property "LCSC" "C72494"
-			(at 378.46 55.88 0)
-			(effects
